File: Schematics/SFB/SFB.kicad_pcb (KiCad board)
At the start: 2 copper layers, 60.3 x 40 mm, 11 parts, among them J1 JST XH 1x5 angled, SW1 SW_DPST, SW2 SW_DPST, SW3 SW_DPST, U1 Arduino_Nano_v3.x, U2 A1326 LUA-T, U3 A1326 LUA-T, U4 A1326 LUA-T, U5 A1326 LUA-T, U6 A1326 LUA-T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

Commit message: Updated; See README.md
Other:
- net class Default removed
- rule pad_to_mask_clearance: 0.051 -> 0
